File: Kicad_Source/fliphackV1.kicad_pcb (KiCad board)
At the start: 2 copper layers, 53 x 76 mm, 60 parts, among them J1 USB_C_Receptacle_USB2.0_14P, J10 SD_Card_Module, J11 1.69 inch IPS TFT LCD Display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, J12 NEO-6M GPS Module, J2 Conn_01x02_Pin, J4 J_NRF24, J6 CC1101_Module, J9 NFC_PN532, Q1 AO3401A, Q2 AO3400A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

Commit message: Add files via upload
Parts:
- J12: value NEO-6M GPS Module -> NEO-8M GPS Module
- SW1: value SW_SP5T_NR01105 -> Button_Switch_SMD:SW-SMD-6P-L10.5-W10.0_C2858290; footprint Button_Switch_THT:SW_NKK_NR01 -> Button_Switch_SMD:SW-SMD-6P-L10.5-W10.0_C2858290
- moved SW1 6.05 mm to (185.5, 144.8)
Connections:
- U1 pad 19: /JOY_OK -> /JOY_DOWN
- U1 pad 31: /JOY_DOWN -> /JOY_L
- U1 pad 32: /JOY_L -> /JOY_R
- U1 pad 33: /JOY_R -> /JOY_OK
Routing:
- net /JOY_OK: track 41.1 -> 49.1 mm
- net GND: track 20.0 -> 16.4 mm, vias 49 -> 51
- net /JOY_DOWN: track 42.5 -> 39.5 mm
- net /JOY_R: track 51.4 -> 50.7 mm
