File: Kicad_Source/fliphackV1.kicad_sch (KiCad schematic)
At the start: 60 parts, among them J1 USB_C_Receptacle_USB2.0_14P, J10 SD_Card_Module, J11 1.69 inch IPS TFT LCD Display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, J12 NEO-6M GPS Module, J2 Conn_01x02_Pin, J4 J_NRF24, J6 CC1101_Module, J9 NFC_PN532, Q1 AO3401A, Q2 AO3400A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

Commit message: Add files via upload
Parts:
- J12: value NEO-6M GPS Module -> NEO-8M GPS Module
- SW1: value SW_SP5T_NR01105 -> Button_Switch_SMD:SW-SMD-6P-L10.5-W10.0_C2858290; footprint Button_Switch_THT:SW_NKK_NR01 -> Button_Switch_SMD:SW-SMD-6P-L10.5-W10.0_C2858290; LCSC C2858286 -> C2858290; MNF PART NUMBER C2858286 -> C2858290
Connections:
- net GND: now also SW1.6 (Common); no longer SW1.C (Common), SW1.MP
- net JOY_DOWN: now also U1.19 (IO11); no longer U1.31 (IO38)
- net JOY_L: now also U1.31 (IO38); no longer U1.32 (IO39)
- net JOY_OK: now also U1.33 (IO40); no longer U1.19 (IO11)
- net JOY_R: now also U1.32 (IO39); no longer U1.33 (IO40)
Changed lines of the file:
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@@
 	)
 	(junction
-		(at 83.82 187.96)
-		(diameter 0)
-		(color 0 0 0 0)
-	)
-	(junction
 		(at 162.56 257.81)
 		(diameter 0)
@@
 	(wire
 		(pts
-			(xy 78.74 187.96) (xy 83.82 187.96)
+			(xy 78.74 185.42) (xy 83.82 185.42)
 		)
 		(stroke
@@
 	(wire
 		(pts
-			(xy 83.82 187.96) (xy 83.82 190.5)
-		)
-		(stroke
-			(width 0)
-			(type default)
-		)
-	)
-	(wire
-		(pts
 			(xy 246.38 133.35) (xy 256.54 133.35)
 		)
@@
 	(wire
 		(pts
-			(xy 83.82 185.42) (xy 83.82 187.96)
-		)
-		(stroke
-			(width 0)
-			(type default)
-		)
-	)
-	(wire
-		(pts
 			(xy 152.4 247.65) (xy 162.56 247.65)
 		)
@@
 	)
 	(label "JOY_OK"
-		(at 205.74 158.75 0)
+		(at 104.14 190.5 0)
 		(effects
 			(font
@@
 		)
 	)
-	(label "JOY_OK"
-		(at 104.14 190.5 0)
+	(label "VBAT"
+		(at 337.82 240.665 0)
 		(effects
 			(font
-				(size 1.27 1.27)
+				(size 1.2446 1.2446)
 			)
 			(justify left bottom)
 		)
 	)
-	(label "VBAT"
-		(at 337.82 240.665 0)
+	(label "JOY_OK"
+		(at 256.54 156.21 0)
 		(effects
 			(font
-				(size 1.2446 1.2446)
+				(size 1.27 1.27)
 			)
 			(justify left bottom)
@@
 		)
 	)
-	(label "JOY_L"
-		(at 256.54 153.67 0)
-		(effects
-			(font
-				(size 1.27 1.27)
-			)
-			(justify left bottom)
-		)
-	)
 	(label "TFT_CS"
 		(at 205.74 171.45 0)
@@
 		)
 	)
-	(label "JOY_R"
-		(at 256.54 156.21 0)
+	(label "CC_GD02"
+		(at 118.11 157.48 0)
 		(effects
 			(font
@@
 		)
 	)
-	(label "CC_GD02"
-		(at 118.11 157.48 0)
+	(label "JOY_R"
+		(at 256.54 153.67 0)
 		(effects
 			(font
@@
 		)
 	)
-	(label "JOY_DOWN"
-		(at 256.54 151.13 0)
-		(effects
-			(font
-				(size 1.27 1.27)
-			)
-			(justify left bottom)
-		)
-	)
 	(label "5V"
 		(at 212.09 264.16 0)
@@
 		)
 	)
+	(label "JOY_L"
+		(at 256.54 151.13 0)
+		(effects
+			(font
+				(size 1.27 1.27)
+			)
+			(justify left bottom)
+		)
+	)
+	(label "JOY_DOWN"
+		(at 205.74 158.75 0)
+		(effects
+			(font
+				(size 1.27 1.27)
+			)
+			(justify left bottom)
+		)
+	)
 	(label "SD_CS"
 		(at 256.54 171.45 0)
@@
 			)
 		)
-		(property "Value" "SW_SP5T_NR01105"
+		(property "Value" "Button_Switch_SMD:SW-SMD-6P-L10.5-W10.0_C2858290"
 			(at 91.44 176.53 0)
 			(effects
@@
 			)
 		)
-		(property "Footprint" "Button_Switch_THT:SW_NKK_NR01"
-			(at 91.44 195.58 0)
+		(property "Footprint" "Button_Switch_SMD:SW-SMD-6P-L10.5-W10.0_C2858290"
+			(at 91.948 198.12 0)
 			(effects
 				(font
@@
 			)
 		)
-		(property "Datasheet" "https://www.nkkswitches.com/pdf/NR01%20Rotaries.pdf"
+		(property "Datasheet" ""
 			(at 91.44 198.12 0)
 			(effects
@@
 			)
 		)
-		(property "Description" "NKK Switches NR01 Series rotary SP5T switch"
-			(at 91.44 185.42 0)
+		(property "Description" "Button_Switch_SMD:SW-SMD-6P-L10.5-W10.0_C2858290"
+			(at 91.948 201.93 0)
 			(effects
 				(font
@@
 			)
 		)
-		(property "MNF PART NUMBER" "C2858286"
-			(at 91.44 194.056 0)
+		(property "MNF PART NUMBER" "C2858290"
+			(at 90.932 195.834 0)
 			(effects
 				(font
@@
 			)
 		)
-		(property "LCSC" "C2858286"
+		(property "LCSC" "C2858290"
 			(at 90.932 193.802 0)
 			(effects
@@
 		(pin "5"
 		)
-		(pin "C"
-		)
 		(pin "4"
 		)
-		(pin "MP"
+		(pin "6"
 		)
 		(pin "3"
@@
 		(lib_name "GND_2")
 		(lib_id "power:GND")
-		(at 78.74 187.96 270)
+		(at 78.74 185.42 270)
 		(unit 1)
 		(exclude_from_sim no)
@@
 		(fields_autoplaced yes)
 		(property "Reference" "#PWR06"
-			(at 72.39 187.96 0)
+			(at 72.39 185.42 0)
 			(effects
 				(font
@@
 		)
 		(property "Value" "GND"
-			(at 74.93 187.9599 90)
+			(at 74.93 185.4199 90)
 			(effects
 				(font
@@
 		)
 		(property "Footprint" ""
-			(at 78.74 187.96 0)
+			(at 78.74 185.42 0)
 			(effects
 				(font
@@
 		)
 		(property "Datasheet" ""
-			(at 78.74 187.96 0)
+			(at 78.74 185.42 0)
 			(effects
 				(font
@@
 		)
 		(property "Description" "Power symbol creates a global label with name \"GND\" , ground"
-			(at 78.74 187.96 0)
+			(at 78.74 185.42 0)
 			(effects
 				(font
@@
 			)
 		)
-		(property "Value" "NEO-6M GPS Module"
+		(property "Value" "NEO-8M GPS Module"
 			(at 55.118 70.866 0)
 			(effects
